File: cutdown.sch (EAGLE design)
At the start: 129 parts, among them J1 RBF_PLUG, Q1 IPB120P04P4L03ATMA1, Q2 SBC817-40LT1G, Q3 SBC817-40LT1G, SW1 M2012LL2W30, U1 ATSAMD21G-A, U2 ATTINY85V-10S, U3 MPL3115A2, U4 R-783.3-0.5_DC-DC, U5 R-783.3-0.5_DC-DC, U6 CD4013B, U7 MC14106BDR2G, X1 ZX62D-B-5PA8, X2 BU-SMA-V, X3 JST-XH-02-PIN-LONG-PAD, X4 JST-XH-02-PIN-LONG-PAD

Commit message: Rev B Hardware
Parts:
- removed C24, C25: 100n, resistor:C-EUC0805
- removed D7: 1N4148, diode:DIODE-SOD323-R
- removed L1: 27n, rcl:L-USL0805
- removed R37, R38, R39, R40, R41, R43, R45, R47: 10.0K, resistor:R-US_R0805
- removed R42, R44, R46: 80.6k, rcl:R-US_R0805
- removed TP10, TP11, TP12, TP13, TP14, TP15, TP16, TP17, TP8, TP9: TPSPAD1-13, testpad:TPSPAD1-13
- removed U$10, U$15: CDBA340L-G, Dector_Parts_TR:CDBA340L-G
- removed U$13: 1053101206, Dector_Parts_TR:1053101206
- removed U$14: MC-146-32.7680KA-A0, Dector_Parts_TR:MC-146-32.7680KA-A0
- removed U$2: DECTOR_PARTS_TR_NANOFIT_1X2_RA, Solar Cell Carrier Board:DECTOR_PARTS_TR_NANOFIT_1X2_RA
- removed U$4: MAX-M8, ubloxLib:MAX-M8
- removed U$6, U$8, U$9: BTS500600-1TEA, Dector_Parts_TR:BTS500600-1TEA
- added D2: 1SMB5913BT3G, 1smb59xx_10:1SMB5913BT3G
- added D3: 1N4148, diode:DIODE-SOD323-R
- added J5: RN114BPC, Dector_Parts_TR:RN114BPC
- added J6: 1053091305, Dector_Parts_TR:1053091305
- added Q5: BTS50060-1TEA, Dector_Parts_TR:BTS50060-1TEA
- added R18, R20: 10.0K, resistor:R-US_R0805
- added R19: 820, rcl:R-US_R0805
- added T1, T2: SBC817-40LT1G, transistor-neu-to92:BC846
- added U10: CAM-M8C-0, Dector_Parts_TR:CAM-M8C-0
- added U8: ATSAMD21G-A, samd21_lib:ATSAMD21G-A
- C1, C4: value 100n -> 10u; device resistor:C-EUC0805 -> rcl:C-EUC1206; MFG AVX -> Samsung; MFG_DESCRIPTION 0.10µF ±10% 25V Ceramic Capacitor X7R 0805 -> CAP CER 10UF 25V X7R 1206; MFG_PN 08053C104KAT2A -> CL31B106KAHZW6E
- C10, C7: device rcl:CPOL-USCT7343 -> rcl:C-EUC1206; MFG (none) -> Samsung; MFG_DESCRIPTION (none) -> CAP CER 10UF 25V X7R 1206; MFG_PN (none) -> CL31B106KAHZW6E; VOLTAGE (none) -> 25V
- C17: value 10n -> 100n; device rcl:C-EUC0805 -> resistor:C-EUC0805; MFG (none) -> AVX; MFG_DESCRIPTION (none) -> 0.10µF ±10% 25V Ceramic Capacitor X7R 0805; MFG_PN (none) -> 08053C104KAT2A; VOLTAGE (none) -> 25V
- C18: value 100n -> 1u; device resistor:C-EUC0805 -> rcl:CPOL-USCT3216; MFG AVX -> Kemet; MFG_DESCRIPTION 0.10µF ±10% 25V Ceramic Capacitor X7R 0805 -> CAP TANT 1UF 10% 16V 1206; MFG_PN 08053C104KAT2A -> T491A105K016AT; VOLTAGE 25V -> (none)
- C19: value 100n -> 22p; device resistor:C-EUC0805 -> rcl:C-EUC0805; MFG AVX -> Kemet; MFG_DESCRIPTION 0.10µF ±10% 25V Ceramic Capacitor X7R 0805 -> CAP CER 22PF 50V C0G/NP0 0805; MFG_PN 08053C104KAT2A -> C0805C220K5GACTU; VOLTAGE 25V -> (none)
- C2: value 1u -> 100n; device rcl:CPOL-USCT3216 -> resistor:C-EUC0805; MFG (none) -> AVX; MFG_DESCRIPTION (none) -> 0.10µF ±10% 25V Ceramic Capacitor X7R 0805; MFG_PN (none) -> 08053C104KAT2A; VOLTAGE (none) -> 25V
- C21: MFG (none) -> Kemet; MFG_DESCRIPTION (none) -> CAP CER 22PF 50V C0G/NP0 0805; MFG_PN (none) -> C0805C220K5GACTU
- C22: value 22p -> 10u; device rcl:C-EUC0805 -> rcl:C-EUC1206; MFG (none) -> Samsung; MFG_DESCRIPTION (none) -> CAP CER 10UF 25V X7R 1206; MFG_PN (none) -> CL31B106KAHZW6E; VOLTAGE (none) -> 25V
- C23: value 10u -> 100n; device rcl:C-EUC1206 -> resistor:C-EUC0805; MFG KEMET -> AVX; MFG_DESCRIPTION 10µF ±5% 25V Ceramic Capacitor X7R 1206 -> 0.10µF ±10% 25V Ceramic Capacitor X7R 0805; MFG_PN C1206X106J3RAC7800 -> 08053C104KAT2A
- C8: value 10u -> 1u; device rcl:CPOL-USCT7343 -> rcl:C-EUC1206; MFG (none) -> KEMET; MFG_DESCRIPTION (none) -> CAP CER 1UF 25V X7R 1206; MFG_PN (none) -> C1206C105K3RACTU; VOLTAGE (none) -> 25V
- C9: value 10u -> 10n; device rcl:CPOL-USCT7343 -> rcl:C-EUC0805; MFG (none) -> Kemet; MFG_DESCRIPTION (none) -> CAP CER 10000PF 50V X7R 0805; MFG_PN (none) -> C0805C103K5RACTU
- D4, D5: value 1SMB5913BT3G -> CDBA340L-G; device 1smb59xx_10:1SMB5913BT3G -> Dector_Parts_TR:CDBA340L-G
- D6: value 1N4148 -> 1SMB5913BT3G; device diode:DIODE-SOD323-R -> 1smb59xx_10:1SMB5913BT3G; MFG Vishay -> (none); MFG_DESCRIPTION DIODE GEN PURP 75V 150MA SOD323 -> (none); MFG_PN 1N4148WS-G3-08 -> (none)
- J1: value RBF_PLUG -> DECTOR_PARTS_TR_NANOFIT_1X2_RA; device SparkFun-Connectors:DB9FEMALE -> Solar Cell Carrier Board:DECTOR_PARTS_TR_NANOFIT_1X2_RA
- LED1, LED2: MFG (none) -> Lite-On; MFG_DESCRIPTION (none) -> LED RED CLEAR SMD; MFG_PN (none) -> LTST-C171KRKT
- LED3, LED4: MFG (none) -> Lite-On; MFG_DESCRIPTION (none) -> LED GREEN CLEAR CHIP SMD; MFG_PN (none) -> LTST-C171GKT
- LS1: MFG (none) -> CUI; MFG_DESCRIPTION (none) -> AUDIO MAGNETIC IND 8-16V TH; MFG_PN (none) -> CEM-1212C
- Q1: value IPB120P04P4L03ATMA1 -> SI2347DS-T1-GE3; device Dector_Parts_TR:IPB120P04P4L03ATMA1 -> Dector_Parts_TR:SI2347DS-T1-GE3; MFG (none) -> Vishay Siliconix; MFG_DESCRIPTION (none) -> MOSFET P-CH 30V 5A SOT-23; MFG_PN (none) -> SI2347DS-T1-GE3
- Q2, Q3: value SBC817-40LT1G -> BTS50060-1TEA; device transistor-neu-to92:BC846 -> Dector_Parts_TR:BTS50060-1TEA; MFG On Semi -> (none); MFG_DESCRIPTION TRANS NPN 45V 0.5A SOT-23 -> (none); MFG_PN SBC817-40LT1G -> (none)
- R1, R11, R13, R25, R26: value 1k -> 10.0K; device rcl:R-US_R0805 -> resistor:R-US_R0805; MFG (none) -> Panasonic; MFG_DESCRIPTION (none) -> RES SMD 10.0K OHM 1% 1/8W 0805; MFG_PN (none) -> ERJ-6ENF1002V; PWR (none) -> 0.125
- R10: value 10.0K -> 80.6k; device resistor:R-US_R0805 -> rcl:R-US_R0805; MFG_DESCRIPTION RES SMD 10.0K OHM 1% 1/8W 0805 -> RES SMD 80.6K OHM 1% 1/8W 0805; MFG_PN ERJ-6ENF1002V -> ERJ-6ENF8062V
- R14: value 820 -> 1k; MFG (none) -> Panasonic; MFG_DESCRIPTION (none) -> RES SMD 1K OHM 1% 1/8W 0805; MFG_PN (none) -> ERJ-6ENF1001V; PWR (none) -> 0.125
- R15: value 10.0K -> 2.00K; MFG_DESCRIPTION RES SMD 10.0K OHM 1% 1/8W 0805 -> RES SMD 2.00K OHM 1% 1/8W 0805; MFG_PN ERJ-6ENF1002V -> ERJ-6ENF2001V
- R2: value 130 -> 80.6k; MFG (none) -> Panasonic; MFG_DESCRIPTION (none) -> RES SMD 80.6K OHM 1% 1/8W 0805; MFG_PN (none) -> ERJ-6ENF8062V; PWR (none) -> 0.125
- R21: value 10.0K -> 130; device resistor:R-US_R0805 -> rcl:R-US_R0805; MFG_DESCRIPTION RES SMD 10.0K OHM 1% 1/8W 0805 -> RES SMD 130 OHM 1% 1/8W 0805; MFG_PN ERJ-6ENF1002V -> ERJ-6ENF1300V
- R22: value 180 -> 130; MFG (none) -> Panasonic; MFG_DESCRIPTION (none) -> RES SMD 130 OHM 1% 1/8W 0805; MFG_PN (none) -> ERJ-6ENF1300V; PWR (none) -> 0.125
- R23, R27, R31, R32, R33: value 10.0K -> 1k; device resistor:R-US_R0805 -> rcl:R-US_R0805; MFG_DESCRIPTION RES SMD 10.0K OHM 1% 1/8W 0805 -> RES SMD 1K OHM 1% 1/8W 0805; MFG_PN ERJ-6ENF1002V -> ERJ-6ENF1001V
- R24: value 100 -> 130; MFG (none) -> Panasonic; MFG_DESCRIPTION (none) -> RES SMD 130 OHM 1% 1/8W 0805; MFG_PN (none) -> ERJ-6ENF1300V; PWR (none) -> 0.125
- R28: value 0 -> 2.00K; device rcl:R-US_R1206 -> resistor:R-US_R0805; MFG (none) -> Panasonic; MFG_DESCRIPTION (none) -> RES SMD 2.00K OHM 1% 1/8W 0805; MFG_PN (none) -> ERJ-6ENF2001V; PWR (none) -> 0.125
- R29: value 0 -> 10.0K; device rcl:R-US_R1206 -> resistor:R-US_R0805; MFG (none) -> Panasonic; MFG_DESCRIPTION (none) -> RES SMD 10.0K OHM 1% 1/8W 0805; MFG_PN (none) -> ERJ-6ENF1002V; PWR (none) -> 0.125
- R3: value 10 -> 10.0K; device rcl:R-US_R0805 -> resistor:R-US_R0805; MFG (none) -> Panasonic; MFG_DESCRIPTION (none) -> RES SMD 10.0K OHM 1% 1/8W 0805; MFG_PN (none) -> ERJ-6ENF1002V; PWR (none) -> 0.125
- R30: value 10.0 -> 10.0K; MFG_DESCRIPTION RES SMD 10.0 OHM 1% 1/8W 0805 -> RES SMD 10.0K OHM 1% 1/8W 0805; MFG_PN ERJ-6ENF10R0V -> ERJ-6ENF1002V
- R34: value 49.9K -> 10.0K; MFG_DESCRIPTION RES SMD 49.9K OHM 1% 1/8W 0805 -> RES SMD 10.0K OHM 1% 1/8W 0805; MFG_PN ERJ-6ENF4992V -> ERJ-6ENF1002V
- R35: value 2.00K -> 220; device resistor:R-US_R0805 -> rcl:R-US_R0805; MFG_DESCRIPTION RES SMD 2.00K OHM 1% 1/8W 0805 -> RES SMD 220 OHM 1% 1/8W 0805; MFG_PN ERJ-6ENF2001V -> ERJ-6ENF2200V
- R36: value 10.0K -> 220; device resistor:R-US_R0805 -> rcl:R-US_R0805; MFG_DESCRIPTION RES SMD 10.0K OHM 1% 1/8W 0805 -> RES SMD 220 OHM 1% 1/8W 0805; MFG_PN ERJ-6ENF1002V -> ERJ-6ENF2200V
- R4: value 130 -> 10.0K; device rcl:R-US_R0805 -> resistor:R-US_R0805; MFG (none) -> Panasonic; MFG_DESCRIPTION (none) -> RES SMD 10.0K OHM 1% 1/8W 0805; MFG_PN (none) -> ERJ-6ENF1002V; PWR (none) -> 0.125
- R5: value 820 -> 49.9K; device rcl:R-US_R0805 -> resistor:R-US_R0805; MFG (none) -> Panasonic; MFG_DESCRIPTION (none) -> RES SMD 49.9K OHM 1% 1/8W 0805; MFG_PN (none) -> ERJ-6ENF4992V; PWR (none) -> 0.125
- R7: value 1k -> 10.0; device rcl:R-US_R0805 -> resistor:R-US_R0805; MFG (none) -> Panasonic; MFG_DESCRIPTION (none) -> RES SMD 10.0 OHM 1% 1/8W 0805; MFG_PN (none) -> ERJ-6ENF10R0V; PWR (none) -> 0.125
- R9: value 10.0K -> 820; device resistor:R-US_R0805 -> rcl:R-US_R0805; MFG_DESCRIPTION RES SMD 10.0K OHM 1% 1/8W 0805 -> RES SMD 820 OHM 1% 1/8W 0805; MFG_PN ERJ-6ENF1002V -> ERJ-6ENF8200V
- SV1: value SAMD21_ISP -> ATTINY_ISP; device con-lstb:MA04-2 -> con-lstb:MA03-2; MFG (none) -> Amphenol; MFG_DESCRIPTION (none) -> CONN HEADER 6POS .100 STR TIN; MFG_PN (none) -> 67996-406HLF
- SV2: value ATTINY_ISP -> SAMD21_ISP; device con-lstb:MA03-2 -> con-lstb:MA04-2; MFG (none) -> Amphenol; MFG_DESCRIPTION (none) -> CONN HEADER 8POS .100 STR TIN; MFG_PN (none) -> 67996-408HLF
- TP2: MFG (none) -> Keystone; MFG_DESCRIPTION (none) -> White PC Test Point, Miniature 0.100 Dia x 0.180 L; MFG_PN (none) -> 5002
- TP7: MFG (none) -> Keystone; MFG_DESCRIPTION (none) -> Black PC Test Point, Miniature 0.100 Dia x 0.180 L; MFG_PN (none) -> 5001
- U1: value ATSAMD21G-A -> R-783.3-0.5_DC-DC; device samd21_lib:ATSAMD21G-A -> Dector_Parts_TR:R-783.3-0.5_DC-DC
- U2: value ATTINY85V-10S -> MC14106BDR2G; device _hhn_attiny25_45_85:ATTINY85V-10S -> Dector_Parts_TR:MC14106BDR2G
- U3: value MPL3115A2 -> CD4013B; device SparkFun-Sensors:MPL3115A2 -> Dector_Parts_TR:CD4013B
- U4: value R-783.3-0.5_DC-DC -> LT1761IS5-3.3; device Dector_Parts_TR:R-783.3-0.5_DC-DC -> Dector_Parts_TR:LT1761IS5-3.3; MFG (none) -> Linear Technology; MFG_DESCRIPTION (none) -> IC REG LIN 3.3V 100MA TSOT23-5; MFG_PN (none) -> LT1761IS5-3.3#TRMPBF
- U5: value R-783.3-0.5_DC-DC -> MCP9700T-E/TT; device Dector_Parts_TR:R-783.3-0.5_DC-DC -> Dector_Parts_TR:MCP9700T-E/TT; MFG (none) -> Microchip Technology; MFG_DESCRIPTION (none) -> SENSOR ANALOG -40C-125C SOT23-3; MFG_PN (none) -> MCP9700T-E/TT
- U6: value CD4013B -> ATTINY85V-10S; device Dector_Parts_TR:CD4013B -> _hhn_attiny25_45_85:ATTINY85V-10S
- U7: value MC14106BDR2G -> MPL3115A2; device Dector_Parts_TR:MC14106BDR2G -> SparkFun-Sensors:MPL3115A2; MFG (none) -> NXP; MFG_DESCRIPTION (none) -> IC ALTIMETER I2C VERSION 8LGA; MFG_PN (none) -> MPL3115A2
- X1: value ZX62D-B-5PA8 -> JST-XH-02-PIN-LONG-PAD; device zx62d-b-5pa8-oshpark_10:ZX62D-B-5PA8 -> Rembrandt Electronics - JST XH Connectors v1-0:JST-XH-02-PIN-LONG-PAD; MFG (none) -> JST Sales America Inc.
- X2: value BU-SMA-V -> JST-XH-02-PIN-LONG-PAD; device con-coax:BU-SMA-V -> Rembrandt Electronics - JST XH Connectors v1-0:JST-XH-02-PIN-LONG-PAD
- X3: value JST-XH-02-PIN-LONG-PAD -> MC-146-32.7680KA-A0; device Rembrandt Electronics - JST XH Connectors v1-0:JST-XH-02-PIN-LONG-PAD -> Dector_Parts_TR:MC-146-32.7680KA-A0
- X4: value JST-XH-02-PIN-LONG-PAD -> ZX62D-B-5PA8; device Rembrandt Electronics - JST XH Connectors v1-0:JST-XH-02-PIN-LONG-PAD -> zx62d-b-5pa8-oshpark_10:ZX62D-B-5PA8
- renumbered U$1 to J2, U$11 to Q4, U$12 to U9, U$3 to J3, U$5 to J4, U$7 to D1
Connections:
- removed net !GPS_RESET!: U$4.9_V_RESET_N, U1.PA19(SER1:3+)
- removed net !OLED_CS!: U1.PB10(SER4:2+), U9.!CS!
- removed net !SAMD21_ARM!: J1.6, R21.2, U1.PB22(SER5:2+)
- removed net 3V3A_VMON: R38.2, R39.1, U1.PA05(AIN5/SER0:1/TC0:1)
- removed net 3V3B_VMON: R40.2, R41.1, U1.PA06(AIN6/SER0:2/TC1:0)
- removed net ATTINY_SCK/!ATTINY_ARM!: J1.7, R17.2, SV2.3, U1.PA11(AIN19/SER0:3+), U2.SCK/SCL/PB2
- removed net BATT1_VMON: R42.1, R43.1, U1.PA07(AIN7/SER0:3/TC1:1)
- removed net BATT2_VMON: R44.1, R45.1, U1.PB02(AIN10/SER5:0)
- removed net GPS_ANTENNA: L1.1, U$4.11_RF_IN, X2.1
- removed net N$25: C21.2, U$14.P4, U1.PA01(XOUT32/SER1:1/TC2:1)
- removed net N$7: D1.A, R42.2, TP6.PP, X3-1.S
- removed net RADIO_GPIO2: U$13.5, U1.PA23(I2C/SER3:0+)
- removed net SQUIB1: J1.8, R5.2, R9.2, U$2.P$1, U$6.OUT
- removed net SQUIB1_GATE: R6.1, U$6.IN, U1.PA14(XIN/SER2:2+)
- removed net SQUIB1_VMON: D4.C, R8.2, R9.1, U1.PA03(AIN1/REFA)
- removed net SQUIB2: J1.9, J3.P$1, R14.2, R15.2, U$8.OUT, U$9.OUT
- removed net SQUIB2_GATE: R10.1, U$8.IN, U1.PA15(XOUT/SER2:3+)
- removed net SQUIB2_GATE_BCKP: R12.1, U$9.IN, U2.PB4
- removed net SQUIB2_VMON: D5.C, R15.1, R16.2, U1.PA04(AIN4/REFB/SER0:0/TC0:0)
- removed net SQUIB_FIRED: R27.1, U1.PB23(SER5:3+), U2.PB3
- removed net VBATT_VMON: R46.2, R47.2, U1.PB03(AIN11/SER5:1)
- new net !SYSTEM_ARM!: J5.TS, R29.2, R30.2, U6.PB3, U8.PA19(SER1:3+)
- new net AREF: U8.PA03(AIN1/REFA)
- new net ATN: U8.PA13(I2C/SER2:1+)
- new net ATTINY_SCK: SV1.3, U6.SCK/SCL/PB2, U8.PA11(AIN19/SER0:3+)
- new net ATTINY_SQUIB_PRI: Q5.IN, R26.1, U6.PB4
- new net BATTPRI: D1.A, R2.2, TP1.PP, X1-1.S
- new net BATTPRI_VMON: R2.1, R3.1, U8.PA02(AIN0/DAC)
- new net BATTSEC: D4.A, R10.2, TP5.PP, X2-1.S
- new net BATTSEC_VMON: R10.1, R11.1, U8.PA07(AIN7/SER0:3/TC1:1)
- new net N$27: C9.2, U4.BYP
- new net N$28: R36.1, U10.26_RXD
- new net RX_LED: U8.PB03(AIN11/SER5:1)
- new net SAMD21_SQUIB_BCKP: Q2.IN, R13.1, U8.PB22(SER5:2+)
- new net SAMD21_SQUIB_PRI: Q3.IN, R20.1, U8.PB23(SER5:3+)
- new net SPARE_GPIO1: J6.4, U8.PB09(AIN3/SER4:1/TC4:1)
- new net SPARE_GPIO2: U8.PA16(I2C/SER1:0+)
- new net SQUIB_BCKP: J1.P$1, J5.R, Q2.OUT, R4.2, R9.2
- new net SQUIB_BCKP_VMON: D2.C, R1.2, R4.1, U8.PA04(AIN4/REFB/SER0:0/TC0:0)
- new net SQUIB_PRI: J3.P$1, J5.S, Q3.OUT, Q5.OUT, R18.2, R19.2
- new net SQUIB_PRI_VMON: D6.C, R17.2, R18.1, U8.PA05(AIN5/SER0:1/TC0:1)
- new net TX_LED: U8.PA27
- new net USB_HOST_EN: U8.PA28
- net !ATTINY_RST!: now also SV1.5, U6.!RESET!/PB5, U8.PA09(I2C/AIN17/SER0:1+); no longer SV2.5, U1.PA09(I2C/AIN17/SER0:1+), U2.!RESET!/PB5
- net !OLED_RES!: now also R34.2, U8.PA14(XIN/SER2:2+); no longer R23.2, U1.PA27
- net !SAMD21_RST!: now also SV2.8, U8.!RESET!; no longer SV1.6, U1.!RESET!
- net 1.2V: now also C18.+, U8.VDDCORE; no longer C2.+, U1.VDDCORE
- net ATTINY_MISO_DO: now also SV1.1, U6.MISO/DO/PB1, U8.PA08(I2C/AIN16/SER0:0+); no longer SV2.1, U1.PA08(I2C/AIN16/SER0:0+), U2.MISO/DO/PB1
- net ATTINY_MOSI_DI: now also SV1.4, U6.MOSI/DI/PB0, U8.PA10(AIN18/SER0:2+); no longer SV2.4, U1.PA10(AIN18/SER0:2+), U2.MOSI/DI/PB0
- net BUZZER: now also R28.2, U8.PA06(AIN6/SER0:2/TC1:0); no longer R22.1, U1.PA16(I2C/SER1:0+)
- net CLK: now also U2C.O, U3A.CLK; no longer TP15.PP, U6A.CLK, U7C.O
- net GND: now also C10.2, C18.-, C19.1, C2.2, C22.2, C7.2, C8.2, D2.A, D6.A, J1.P$2, J5.T, J6.5, Q2.GND, Q3.GND, Q5.GND, R11.2, R13.2, R14.1, R16.2, R20.2, R23.1, R25.2, R26.2, R27.1, R3.2, R7.2, SV1.6, SV2.1, SV2.2, SV2.3, SV2.4, T1.E, T2.E, TP7.PP, U1.GND, U10.10_GND, U10.11_GND, U10.12_GND, U10.13_GND, U10.14_GND, U10.15_GND, U10.18_GND, U10.19_GND, U10.21_GND, U10.22_GND, U10.27_GND, U10.31_GND, U10.4_GND, U10.5_GND, U2D.I, U2E.I, U2F.I, U2P.GND, U3A.D, U3A.RESET, U3B.CLK, U3B.D, U3B.RESET, U3B.SET, U3P.GND, U6.GND, U7.GND, U8.GND@18, U8.GND@35, U8.GND@42, U8.GNDANA, U9.!CS!, X1-2.S, X2-2.S, X4G$1.5; no longer C10.-, C18.2, C19.2, C2.-, C22.1, C24.2, C25.2, C7.-, C8.-, C9.-, D4.A, D5.A, J1.1, J1.2, J1.3, J1.4, J1.5, Q2.E, Q3.E, R10.2, R11.1, R12.2, R13.1, R27.2, R28.1, R28.2, R29.1, R29.2, R30.2, R36.2, R37.2, R39.2, R41.2, R43.2, R45.2, R47.1, R6.2, R7.1, SV1.1, SV1.2, SV1.3, SV1.4, SV2.6, TP10.PP, TP11.PP, TP13.PP, TP5.PP, TP9.PP, U$13.6, U$2.P$2, U$4.10_GND, U$4.12_GND, U$4.1_GND, U$6.GND, U$8.GND, U$9.GND, U1.GND@18, U1.GND@35, U1.GND@42, U1.GNDANA, U2.GND, U3.GND, U6A.D, U6A.RESET, U6B.CLK, U6B.D, U6B.RESET, U6B.SET, U6P.GND, U7D.I, U7E.I, U7F.I, U7P.GND, X1G$1.5, X2.2, X3-2.S, X4-2.S
- net GPS_RX: now also R36.2, U8.PA18(SER1:2+); no longer U$4.3_RXD, U1.PA18(SER1:2+)
- net GPS_TX: now also R35.2, U8.PA17(I2C/SER1:1+); no longer U$4.2_TXD, U1.PA17(I2C/SER1:1+)
- net HEATER_GATE: now also U8.PA15(XOUT/SER2:3+); no longer U1.PA28
- net N$1: now also D5.A; no longer TP8.PP, U$15.A
- net N$10: now also U10.16_RF_OUT, U10.17_RF_IN; no longer C17.1, L1.2, R3.1
- net N$11: now also R35.1, U10.25_TXD; no longer R3.2, U$4.14_VCC_RF
- net N$12: now also C21.2, U8.PA01(XOUT32/SER1:1/TC2:1), X3.P4; no longer R44.2, TP7.PP, U$10.A, X4-1.S
- net N$13: now also LED3.A, R21.1; no longer LED1.A, R2.1
- net N$14: now also Q2.IS, R14.2; no longer R7.2, U$6.IS
- net N$15: now also LED4.A, R22.1; no longer LED2.A, R4.1
- net N$16: now also LED1.A, R9.1; no longer LED3.A, R5.1
- net N$17: now also R8.1, U3A.!Q; no longer R32.1, TP12.PP, U6A.Q
- net N$18: now also U2B.O, U2C.I; no longer U7B.O, U7C.I
- net N$19: now also Q3.IS, R23.2; no longer R11.2, U$8.IS
- net N$2: now also R28.1, T2.B; no longer Q3.B, R22.2
- net N$20: now also Q5.IS, R27.2; no longer R13.2, U$9.IS
- net N$21: now also LED2.A, R19.1; no longer LED4.A, R14.1
- net N$23: now also R25.1; no longer R37.1
- net N$24: now also C19.2, U8.PA00(XIN32/SER1:0/TC2:0), X3.P1; no longer C22.2, U$14.P1, U1.PA00(XIN32/SER1:0/TC2:0)
- net N$26: now also LS1.2, T2.C; no longer D7.A, LS1.1, Q3.C
- net N$3: now also R7.1; no longer R30.1
- net N$4: now also R6.2, R8.2; no longer R31.2, R32.2
- net N$5: now also C7.1, D3.A, R5.2, U2A.I; no longer C23.1, D6.A, R34.2, U7A.I
- net N$6: now also R15.1, T1.B; no longer Q2.B, R35.1
- net N$8: now also R12.2, T1.C, U2B.I; no longer Q2.C, R33.2, U7B.I
- net N$9: now also C13.1, U7.CAP; no longer C19.1, U3.CAP
- net OLED_MISO: now also U8.PA12(I2C/SER2:0+); no longer U1.PB09(AIN3/SER4:1/TC4:1)
- net OLED_MOSI: now also U8.PB10(SER4:2+); no longer U1.PB08(AIN2/SER4:0/TC4:0)
- net OLED_SCLK: now also U8.PB11(SER4:3+); no longer U1.PB11(SER4:3+)
- net PRESSURE_SCL: now also R32.1, U7.SCL, U8.PA23(I2C/SER3:0+); no longer R25.1, U1.PA13(I2C/SER2:1+), U3.SCL
- net PRESSURE_SDA: now also R33.1, U7.SDA, U8.PA22(I2C/SER3:0+); no longer R26.1, U1.PA12(I2C/SER2:0+), U3.SDA
- net PWR_OFF: now also R15.2, R16.1, U8.PB08(AIN2/SER4:0/TC4:0); no longer R35.2, R36.1, U1.PA22(I2C/SER3:0+)
- net RADIO_RX: now also J6.3, U8.PA20(SER5:2+); no longer U$13.3, U1.PA20(SER5:2+)
- net RADIO_TX: now also J6.2, U8.PA21(SER5:3+); no longer U$13.2, U1.PA21(SER5:3+)
- net SAMD21_SWCLK: now also R31.1, SV2.7, U8.PA30(SWCLK/SER1:2+); no longer R1.1, SV1.7, U1.PA30(SWCLK/SER1:2+)
- net SAMD21_SWDIO: now also SV2.5, U8.PA31(SWDIO/SER1:3+); no longer SV1.5, U1.PA31(SWDIO/SER1:3+)
- net SET: now also U2A.O, U3A.SET; no longer TP16.PP, U6A.SET, U7A.O
- net THERMISTOR_VOUT: now also U5.VOUT, U8.PB02(AIN10/SER5:0); no longer U1.PA02(AIN0/DAC)
- net USB_D+: now also U8.PA25(SER3:3+), X4G$1.3; no longer U1.PA25(SER3:3+), X1G$1.3
- net USB_D-: now also U8.PA24(SER3:2+), X4G$1.2; no longer U1.PA24(SER3:2+), X1G$1.2
- net VBATT_RAW: now also D4.C, D5.C, TP2.PP; no longer TP17.PP, U$10.C, U$15.C
- net VCC_1: now also C14.1, C15.1, C17.1, C22.1, C23.1, J6.1, R1.1, R17.1, R21.2, R30.1, R31.2, R32.2, R33.2, R34.1, SV2.6, TP4.PP, U1.VOUT, U10.1_VCC_IO, U10.8_V_BCKP, U10.9_VCC, U5.VDD, U7.VDD, U7.VDDIO, U8.VDDANA, U8.VDDIN, U8.VDDIO@17, U8.VDDIO@36; no longer C10.+, C18.1, C5.1, C6.1, D7.C, LS1.2, R1.2, R16.1, R2.2, R21.1, R23.1, R25.2, R26.2, R38.1, R8.1, SV1.8, TP1.PP, U$4.7_VCC_IO, U$4.8_VCC, U1.VDDANA, U1.VDDIN, U1.VDDIO@17, U1.VDDIO@36, U3.VDD, U3.VDDIO, U4.VOUT
- net VCC_2: now also C10.1, C11.1, C9.1, R22.2, R29.1, SV1.2, TP6.PP, U4.VOUT, U6.VCC; no longer C1.1, C14.1, C15.1, C8.+, R17.1, R4.2, R40.1, SV2.2, TP2.PP, U$13.1, U$4.6_V_BCKP, U2.VCC, U5.VOUT
- net VSW: now also C5.1, C6.1, D3.C, R12.1, R5.1, R6.1, U2P.VDD, U3P.VDD; no longer C24.1, C25.1, D6.C, R31.1, R33.1, R34.1, TP14.PP, U6P.VDD, U7P.VDD
- net V_BATT: now also C1.1, C2.1, C8.1, LS1.1, Q2.VS, Q3.VS, Q5.VS, U1.VIN, U4.!SHDN; no longer C11.1, C13.1, C7.+, C9.+, R46.1, TP4.PP, U$6.VS, U$8.VS, U$9.VS, U5.VIN
- net V_USB: now also X4G$1.1; no longer X1G$1.1
Other:
- note added: "30V, 5A, 0.042 ohm"
- note added: "Backup Squib Circuit"
- note added: "BattPri"
- note added: "BattSec"
- note added: "Bootloader"
- note added: "D"
- note added: "G"
- note added: "LDO will have low efficiency, but only powers ATtiny at <1mA, so the little extra generated heat will be small"
- note added: "Primary Squib Backup MCU Circuit"
- note added: "Primary Squib Circuit"
- note added: "S"
- note added: "Squibs shorted out when RBF plug connected"
- note added: "Switches short when removed"
- note added: "decrease UART switching noise by addition of resistors"
- note added: "u-blox CAM-M8C GPS Receiver + Antenna"
- note removed: "40V, 100A, 0.003 ohm"
- note removed: "Batt1"
- note removed: "Batt2"
- note removed: "Each signal shorted to GND in plug"
- note removed: "SER5:0"
- note removed: "SER5:1"
- note removed: "Squib 1 circuit"
- note removed: "Squib 2 backup circuit"
- note removed: "Squib 2 circuit"
- note removed: "Squibs shorted out when RBF DB9 is connected"
- note removed: "TCC0:WO[6]"
- note removed: "Todo: oscillator?"
- note removed: "u-blox MAX-M8C GPS Receiver"
- moved on the sheet: C1, C11, C12, C13, C14, C15, C16, C17, C19, C22, C23, C3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

Commit message: Rev D files
Parts:
- removed C6: 100n, resistor:C-EUC0805
- removed C7: 10u, rcl:C-EUC1206
- removed SW1: M2012LL2W30, Dector_Parts_TR:M2012LL2W30_SPDT_SW
- removed T1: SBC817-40LT1G, transistor-neu-to92:BC846
- removed TP1, TP2, TP5: TPSPAD1-13, testpad:TPSPAD1-13
- removed U3: CD4013B, Dector_Parts_TR:CD4013B
- removed X1, X2: JST-XH-02-PIN-LONG-PAD, Rembrandt Electronics - JST XH Connectors v1-0:JST-XH-02-PIN-LONG-PAD
- added J7: 1053141208, Dector_Parts_TR:1053141208
- added PB1: FP11SPA1B1TP03, Dector_Parts_TR:FP11SPA1B1TP03
- added Q6: SI2347DS-T1-GE3, Dector_Parts_TR:SI2347DS-T1-GE3
- added R37, R38, R39: 2, resistor:R-US_R2512
- added R40, R41: 80.6k, rcl:R-US_R0805
- added R42, R43: 10.0K, resistor:R-US_R0805
- D3: value 1N4148 -> BAT54HT1G; device diode:DIODE-SOD323-R -> Dector_Parts_TR:BAT54HT1G; MFG Vishay -> ON Semiconductor; MFG_DESCRIPTION DIODE GEN PURP 75V 150MA SOD323 -> DIODE SCHOTTKY 30V 200MA SOD323; MFG_PN 1N4148WS-G3-08 -> BAT54HT1G
- D5: value CDBA340L-G -> BAT54HT1G; device Dector_Parts_TR:CDBA340L-G -> Dector_Parts_TR:BAT54HT1G; MFG (none) -> ON Semiconductor; MFG_DESCRIPTION (none) -> DIODE SCHOTTKY 30V 200MA SOD323; MFG_PN (none) -> BAT54HT1G
- J2: value 1053091304 -> S4B-XH-SM4-TB-3S-BALANCE; device Dector_Parts_TR:1053091304 -> Dector_Parts_TR:S4B-XH-SM4-TB-3S-BALANCE; MFG (none) -> JST Sales America Inc.; MFG_DESCRIPTION (none) -> CONN HEADER SMD R/A 4POS 2.5MM; MFG_PN (none) -> S4B-XH-SM4-TB(LF)(SN)
- J4: value 1053101206 -> S4B-XH-SM4-TB-3S-BALANCE; device Dector_Parts_TR:1053101206 -> Dector_Parts_TR:S4B-XH-SM4-TB-3S-BALANCE; MFG (none) -> JST Sales America Inc.; MFG_DESCRIPTION (none) -> CONN HEADER SMD R/A 4POS 2.5MM; MFG_PN (none) -> S4B-XH-SM4-TB(LF)(SN)
- LS1: value BUZZER-PTH_KIT -> CEM-1212C; device SparkFun-Electromechanical:BUZZER-PTH_KIT -> Dector_Parts_TR:CEM-1212C; MFG CUI -> CUI Devices
- R12, R16, R6, R8: value 10.0K -> 2; device resistor:R-US_R0805 -> resistor:R-US_R2512; MFG Panasonic -> Bourns Inc.; MFG_DESCRIPTION RES SMD 10.0K OHM 1% 1/8W 0805 -> RES SMD 2 OHM 5% 2W 2512; MFG_PN ERJ-6ENF1002V -> CRM2512-JW-2R0ELF; PWR 0.125 -> 2
- R15: value 2.00K -> 2; device resistor:R-US_R0805 -> resistor:R-US_R2512; MFG Panasonic -> Bourns Inc.; MFG_DESCRIPTION RES SMD 2.00K OHM 1% 1/8W 0805 -> RES SMD 2 OHM 5% 2W 2512; MFG_PN ERJ-6ENF2001V -> CRM2512-JW-2R0ELF; PWR 0.125 -> 2
- R5: value 49.9K -> 2; device resistor:R-US_R0805 -> resistor:R-US_R2512; MFG Panasonic -> Bourns Inc.; MFG_DESCRIPTION RES SMD 49.9K OHM 1% 1/8W 0805 -> RES SMD 2 OHM 5% 2W 2512; MFG_PN ERJ-6ENF4992V -> CRM2512-JW-2R0ELF; PWR 0.125 -> 2
- R7: value 10.0 -> 2; device resistor:R-US_R0805 -> resistor:R-US_R2512; MFG Panasonic -> Bourns Inc.; MFG_DESCRIPTION RES SMD 10.0 OHM 1% 1/8W 0805 -> RES SMD 2 OHM 5% 2W 2512; MFG_PN ERJ-6ENF10R0V -> CRM2512-JW-2R0ELF; PWR 0.125 -> 2
- U2: value MC14106BDR2G -> LTC2955ITS8-2; device Dector_Parts_TR:MC14106BDR2G -> Dector_Parts_TR:LTC2955ITS8-2; MFG (none) -> Linear Technology/Analog Devices; MFG_DESCRIPTION (none) -> IC CTLR ON/OFF PUSHBUTT TSOT23-8; MFG_PN (none) -> LTC2955ITS8-2#TRMPBF
Connections:
- removed net CLK: U2C.O, U3A.CLK
- removed net N$1: D5.A, J2.1, J2.2
- removed net PWR_OFF: R15.2, R16.1, U8.PB08(AIN2/SER4:0/TC4:0)
- removed net SET: U2A.O, U3A.SET
- removed net VBATT_RAW: D1.C, D4.C, D5.C, SW1.1, TP2.PP
- removed net VSW: C5.1, C6.1, D3.C, Q1.S, R12.1, R5.1, R6.1, SW1.2, U2P.VDD, U3P.VDD
- new net !BATT_EN: R40.1, R41.1, U2.!EN
- new net !PWR_OFF!: R43.1, U2.!KILL, U8.PB08(AIN2/SER4:0/TC4:0)
- new net BATTPRI_1S: J2.1S, J7.3
- new net BATTPRI_2S: J2.2S, J7.2
- new net BATTPRI_RAW: D3.A, J2.VBAT/3S, J7.1, Q1.S
- new net BATTSEC_1S: J4.1S, J7.7
- new net BATTSEC_2S: J4.2S, J7.8
- new net BATTSEC_RAW: D5.A, J4.VBAT/3S, J7.4, Q6.S
- new net N$25: R38.1, R39.2
- new net N$29: Q4.D6, Q4.D@1, Q4.D@2, Q4.D@5, R39.1
- new net N$30: Q6.G, R41.2
- new net N$32: PB1.3, U2.!PB
- new net N$33: C5.1, D3.C, D5.C, U2.V_IN
- new net N$7: R12.1, R8.2
- net !SAMD21_RST!: now also R42.1, U2.!INT
- net BATTPRI: now also Q1.D; no longer TP1.PP, X1-1.S
- net BATTSEC: now also Q6.D; no longer TP5.PP, X2-1.S
- net GND: now also J2.GND, J4.GND, J7.5, J7.6, PB1.1, U2.GND, U2.ON; no longer C6.2, C7.2, J2.3, J2.4, J4.3, J4.5, R16.2, R7.2, T1.E, U2D.I, U2E.I, U2F.I, U2P.GND, U3A.D, U3A.RESET, U3B.CLK, U3B.D, U3B.RESET, U3B.SET, U3P.GND, X1-2.S, X2-2.S
- net N$17: now also R15.1, R16.2; no longer R8.1, U3A.!Q
- net N$18: now also R16.1, R37.2; no longer U2B.O, U2C.I
- net N$22: now also R37.1, R38.2; no longer J4.6, Q4.D6, Q4.D@1, Q4.D@2, Q4.D@5
- net N$26: now also LS1.-; no longer LS1.2
- net N$3: now also R5.2, R6.1; no longer R7.1, SW1.3
- net N$4: now also R40.2; no longer R6.2, R8.2
- net N$5: now also R6.2, R7.1; no longer C7.1, D3.A, R5.2, U2A.I
- net N$6: now also R7.2, R8.1; no longer R15.1, T1.B
- net N$8: now also R15.2; no longer T1.C, U2B.I
- net THERMISTOR_VOUT: no longer J4.2
- net VCC_1: now also R42.2, R43.2; no longer J4.1
- net V_BATT: now also D1.C, D4.C, LS1.+, R5.1; no longer J4.4, LS1.1, Q1.D
Other:
- note added: "20 Ohm eq. heater array => 0.65 A max => 0.845 W max/resistor Resistors are 2W rated"
- note added: "BattPri Balance Connector"
- note added: "BattSec Balance Connector"
- note added: "Battery & Charge Connectors"
- note added: "Battery Charge Connector / Ground Power Connector"
- note added: "Battery Diode Or"
- note added: "Battery Switches"
- note added: "Battery Voltage Monitors"
- note added: "Pushbutton On/Off Controller"
- note removed: "(Locking Lever)"
- note removed: "A"
- note removed: "BattPri"
- note removed: "BattSec"
- note removed: "Batteries"
- note removed: "Battery Discharge Protection Circuit"
- note removed: "Battery Switch"
- note removed: "G"
- note removed: "High turns on Q3"
- note removed: "OFF = High then a 50 msec Low"
- note removed: "Power supply connector (For testing/configuring)"
- note removed: "RUN = Low or High Z"
- note removed: "S"
- note removed: "Unused Gates"
- moved on the sheet: C1, C10, C2, C3, C4, C5, C8, C9, D1, D4, D5, Q1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
